File: BME68x Adaptor.kicad_pcb (KiCad board)
At the start: 2 copper layers, 20 x 20 mm, 7 parts, among them J1 Conn_01x06, U1 BME680

Commit message: layout finished
Parts:
- moved C1 5.00 mm to (142.6, 92.0)
- moved R1 2.60 mm to (137.4, 92.0)
- moved R2 2.60 mm to (134.8, 92.0)
- moved R3 2.60 mm to (140.0, 92.0)
- moved J1 0.47 mm to (146.3, 98.6)
- moved C2 0.10 mm to (145.2, 92.0)
Routing:
- net +3V3: track 43.4 -> 49.7 mm, vias 5 -> 4
- net GND: track 6.01 -> 7.04 mm
Other:
- board text added: "1"
- board text added: "BME680"
- board text added: "BME688"
- board text added: "BME68X ADAPTOR 1.0 LC APR 2022"
- board text added: "JLCJLCJLCJLC"

Commit message: Silkscreen improved
Parts:
- moved J1 0.35 mm to (146.3, 98.2)
Other:
- board text added: "ADAPTOR"
- board text added: "BME68X"
